File: board/minimal/TurtlePico-Minimal.kicad_sch (KiCad schematic)
At the start: 0 parts

Commit message: change core to rp2350b and some pin out
Other:
- sheet RP2040 renamed RP2350B
- sheet RP2350B: file RP2040.kicad_sch -> RP2350B.kicad_sch
