File: board/minimal/Audio.kicad_sch (KiCad schematic)
At the start: 12 parts, among them J9 AudioJack3, U10 PCM5102A

Commit message: set footprint
Parts:
- renumbered C37 to C36, C38 to C37, C32 to C38, C33 to C40, C34 to C41, C35 to C42, C36 to C43, J9 to J10, R22 to R24, U10 to U9
Changed lines of the file:
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@@
 		(on_board yes)
 		(dnp no)
-		(property "Reference" "C37"
+		(property "Reference" "C36"
 			(at 128.27 103.505 0)
 			(effects
@@
 			(project "TurtlePico-Minimal"
 				(path "/7af2d99d-e350-48e7-86b4-20911ea922f3/c005a3df-ded2-48f6-91de-22e6372e232d"
-					(reference "C37")
+					(reference "C36")
 					(unit 1)
 				)
@@
 		(dnp no)
 		(fields_autoplaced yes)
-		(property "Reference" "#PWR051"
+		(property "Reference" "#PWR061"
 			(at 177.8 102.87 0)
 			(hide yes)
@@
 			(project "TurtlePico-Minimal"
 				(path "/7af2d99d-e350-48e7-86b4-20911ea922f3/c005a3df-ded2-48f6-91de-22e6372e232d"
-					(reference "#PWR051")
+					(reference "#PWR061")
 					(unit 1)
 				)
@@
 		(on_board yes)
 		(dnp no)
-		(property "Reference" "R22"
+		(property "Reference" "R24"
 			(at 135.89 94.615 90)
 			(effects
@@
 			(project "TurtlePico-Minimal"
 				(path "/7af2d99d-e350-48e7-86b4-20911ea922f3/c005a3df-ded2-48f6-91de-22e6372e232d"
-					(reference "R22")
+					(reference "R24")
 					(unit 1)
 				)
@@
 		(on_board yes)
 		(dnp no)
-		(property "Reference" "C33"
+		(property "Reference" "C40"
 			(at 142.24 100.965 0)
 			(effects
@@
 			(project "TurtlePico-Minimal"
 				(path "/7af2d99d-e350-48e7-86b4-20911ea922f3/c005a3df-ded2-48f6-91de-22e6372e232d"
-					(reference "C33")
+					(reference "C40")
 					(unit 1)
 				)
@@
 		(on_board yes)
 		(dnp no)
-		(property "Reference" "C35"
+		(property "Reference" "C42"
 			(at 177.8 102.235 0)
 			(effects
@@
 			(project "TurtlePico-Minimal"
 				(path "/7af2d99d-e350-48e7-86b4-20911ea922f3/c005a3df-ded2-48f6-91de-22e6372e232d"
-					(reference "C35")
+					(reference "C42")
 					(unit 1)
 				)
@@
 		(on_board yes)
 		(dnp no)
-		(property "Reference" "C32"
+		(property "Reference" "C38"
 			(at 137.16 100.965 0)
 			(effects
@@
 			(project "TurtlePico-Minimal"
 				(path "/7af2d99d-e350-48e7-86b4-20911ea922f3/c005a3df-ded2-48f6-91de-22e6372e232d"
-					(reference "C32")
+					(reference "C38")
 					(unit 1)
 				)
@@
 		(dnp no)
 		(fields_autoplaced yes)
-		(property "Reference" "#PWR050"
+		(property "Reference" "#PWR059"
 			(at 119.38 91.44 0)
 			(hide yes)
@@
 			(project "TurtlePico-Minimal"
 				(path "/7af2d99d-e350-48e7-86b4-20911ea922f3/c005a3df-ded2-48f6-91de-22e6372e232d"
-					(reference "#PWR050")
+					(reference "#PWR059")
 					(unit 1)
 				)
@@
 		(on_board yes)
 		(dnp no)
-		(property "Reference" "#PWR052"
+		(property "Reference" "#PWR062"
 			(at 177.8 115.57 0)
 			(hide yes)
@@
 			(project "TurtlePico-Minimal"
 				(path "/7af2d99d-e350-48e7-86b4-20911ea922f3/c005a3df-ded2-48f6-91de-22e6372e232d"
-					(reference "#PWR052")
+					(reference "#PWR062")
 					(unit 1)
 				)
@@
 		(on_board yes)
 		(dnp no)
-		(property "Reference" "U10"
+		(property "Reference" "U9"
 			(at 121.3359 87.63 0)
 			(effects
@@
 			(project "TurtlePico-Minimal"
 				(path "/7af2d99d-e350-48e7-86b4-20911ea922f3/c005a3df-ded2-48f6-91de-22e6372e232d"
-					(reference "U10")
+					(reference "U9")
 					(unit 1)
 				)
@@
 		(on_board yes)
 		(dnp no)
-		(property "Reference" "#PWR054"
+		(property "Reference" "#PWR060"
 			(at 144.78 128.27 0)
 			(hide yes)
@@
 			(project "TurtlePico-Minimal"
 				(path "/7af2d99d-e350-48e7-86b4-20911ea922f3/c005a3df-ded2-48f6-91de-22e6372e232d"
-					(reference "#PWR054")
+					(reference "#PWR060")
 					(unit 1)
 				)
@@
 		(on_board yes)
 		(dnp no)
-		(property "Reference" "C34"
+		(property "Reference" "C41"
 			(at 171.45 102.235 0)
 			(effects
@@
 			(project "TurtlePico-Minimal"
 				(path "/7af2d99d-e350-48e7-86b4-20911ea922f3/c005a3df-ded2-48f6-91de-22e6372e232d"
-					(reference "C34")
+					(reference "C41")
 					(unit 1)
 				)
@@
 		(on_board yes)
 		(dnp no)
-		(property "Reference" "C36"
+		(property "Reference" "C43"
 			(at 184.15 102.235 0)
 			(effects
@@
 			(project "TurtlePico-Minimal"
 				(path "/7af2d99d-e350-48e7-86b4-20911ea922f3/c005a3df-ded2-48f6-91de-22e6372e232d"
-					(reference "C36")
+					(reference "C43")
 					(unit 1)
 				)
@@
 		(on_board yes)
 		(dnp no)
-		(property "Reference" "C38"
+		(property "Reference" "C37"
 			(at 133.35 118.11 90)
 			(effects
@@
 			(project "TurtlePico-Minimal"
 				(path "/7af2d99d-e350-48e7-86b4-20911ea922f3/c005a3df-ded2-48f6-91de-22e6372e232d"
-					(reference "C38")
+					(reference "C37")
 					(unit 1)
 				)
@@
 		(on_board yes)
 		(dnp no)
-		(property "Reference" "J9"
+		(property "Reference" "J10"
 			(at 155.321 91.694 0)
 			(effects
@@
 			(project "TurtlePico-Minimal"
 				(path "/7af2d99d-e350-48e7-86b4-20911ea922f3/c005a3df-ded2-48f6-91de-22e6372e232d"
-					(reference "J9")
+					(reference "J10")
 					(unit 1)
 				)
@@
 		(on_board yes)
 		(dnp no)
-		(property "Reference" "#PWR053"
+		(property "Reference" "#PWR058"
 			(at 102.87 128.27 0)
 			(hide yes)
@@
 			(project "TurtlePico-Minimal"
 				(path "/7af2d99d-e350-48e7-86b4-20911ea922f3/c005a3df-ded2-48f6-91de-22e6372e232d"
-					(reference "#PWR053")
-					(unit 1)
-				)
+					(reference "#PWR058")
+					(unit 1)
+				)
