File: board/minimal/LED_Switch.kicad_sch (KiCad schematic)
At the start: 14 parts, among them J10 LED, J11 LED, Q3 2SC4213, Q4 2SC4213, SW3 SW_{R}, SW4 SW_{L}, SW5 SW_DIP_x03

Commit message: edit schematics
Parts:
- removed RV1: 10k, Potentiometer_SMD:Potentiometer_ACP_CA6-VSMD_Vertical, symbol Device:R_Potentiometer
Changed lines of the file:
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@@
   (junction (at 187.96 109.22) (diameter 0) (color 0 0 0 0)
   )
-  (junction (at 160.02 107.95) (diameter 0) (color 0 0 0 0)
-  )
   (junction (at 144.78 119.38) (diameter 0) (color 0 0 0 0)
   )
-  (wire (pts (xy 168.91 113.03) (xy 170.18 113.03))
-    (stroke (width 0) (type default))
-  )
-  (wire (pts (xy 160.02 116.84) (xy 165.1 116.84))
-    (stroke (width 0) (type default))
-  )
   (wire (pts (xy 127 95.25) (xy 144.78 95.25))
     (stroke (width 0) (type default))
@@
     (stroke (width 0) (type default))
   )
-  (wire (pts (xy 160.02 107.95) (xy 160.02 116.84))
-    (stroke (width 0) (type default))
-  )
   (wire (pts (xy 187.96 111.76) (xy 190.5 111.76))
     (stroke (width 0) (type default))
@@
     (stroke (width 0) (type default))
   )
-  (wire (pts (xy 172.72 116.84) (xy 179.07 116.84))
-    (stroke (width 0) (type default))
-  )
   (wire (pts (xy 133.35 110.49) (xy 133.35 111.76))
     (stroke (width 0) (type default))
@@
     (effects (font (size 1.27 1.27)) (justify left))
     (property "Intersheetrefs" "${INTERSHEET_REFS}" (at 217.6514 109.22 0)
-      (effects (font (size 1.27 1.27)) (justify left) hide)
-    )
-  )
-  (global_label "Volume" (shape output) (at 170.18 113.03 0) (fields_autoplaced)
-    (effects (font (size 1.27 1.27)) (justify left))
-    (property "Intersheetrefs" "${INTERSHEET_REFS}" (at 179.9989 113.03 0)
       (effects (font (size 1.27 1.27)) (justify left) hide)
     )
@@
         (path "/7af2d99d-e350-48e7-86b4-20911ea922f3/3559871a-0f23-4a86-a659-f5f50e9db57b"
           (reference "Q3") (unit 1)
-        )
-      )
-    )
-  )
-  (symbol (lib_id "Device:R_Potentiometer") (at 168.91 116.84 90) (unit 1)
-    (in_bom yes) (on_board yes) (dnp no)
-    (property "Reference" "RV1" (at 167.64 119.38 90)
-      (effects (font (size 1.27 1.27)) (justify right))
-    )
-    (property "Value" "10k" (at 167.64 116.84 90)
-      (effects (font (size 1.27 1.27)) (justify right))
-    )
-    (property "Footprint" "Potentiometer_SMD:Potentiometer_ACP_CA6-VSMD_Vertical" (at 168.91 116.84 0)
-      (effects (font (size 1.27 1.27)) hide)
-    )
-    (property "Datasheet" "~" (at 168.91 116.84 0)
-      (effects (font (size 1.27 1.27)) hide)
-    )
-    (pin "2")
-    (pin "3")
-    (pin "1")
-    (instances
-      (project "TurtlePico-Minimal"
-        (path "/7af2d99d-e350-48e7-86b4-20911ea922f3/3559871a-0f23-4a86-a659-f5f50e9db57b"
-          (reference "RV1") (unit 1)
         )
       )
@@
         )
       )
-    )
-  )
-  (symbol (lib_id "power:GND") (at 179.07 116.84 0) (unit 1)
-    (in_bom yes) (on_board yes) (dnp no)
-    (property "Reference" "#PWR058" (at 179.07 123.19 0)
-      (effects (font (size 1.27 1.27)) hide)
-    )
-    (property "Value" "GND" (at 182.118 118.872 0)
-      (effects (font (size 1.27 1.27)))
-    )
-    (property "Footprint" "" (at 179.07 116.84 0)
-      (effects (font (size 1.27 1.27)) hide)
-    )
-    (property "Datasheet" "" (at 179.07 116.84 0)
-      (effects (font (size 1.27 1.27)) hide)
-    )
-    (pin "1")
-    (instances
-      (project "TurtlePico-Minimal"
-        (path "/7af2d99d-e350-48e7-86b4-20911ea922f3/3559871a-0f23-4a86-a659-f5f50e9db57b"
-          (reference "#PWR058") (unit 1)
-        )
-      )

Commit message: add some connectors
Parts:
- removed SW5: SW_DIP_x03, DS04254203BKSMT:DS04254203BKSMT, symbol Switch:SW_DIP_x03
- added RV1: 50k, symbol Device:R_Potentiometer
- added SW5: SW_DIP_x04, symbol Switch:SW_DIP_x04
Connections:
- net +3.3V: now also RV1.1, SW5.1, SW5.2, SW5.3, SW5.4
- net GND: now also RV1.3
- net SW_{DIP}1: now also SW5.8
- net SW_{DIP}2: now also SW5.7
- net SW_{DIP}3: now also SW5.6
- new net SW_{DIP}4: SW5.5
- new net Volume: RV1.2

Commit message: set footprint
Parts:
- RV1: footprint (none) -> Potentiometer_THT:Potentiometer_Bourns_3339P_Vertical_HandSoldering
- SW5: footprint (none) -> Package_DIP:DIP-8_W7.62mm
- renumbered D4 to D3, D3 to D4, J10 to J11, J11 to J12, Q3 to Q2, Q4 to Q3, R27 to R25, R24 to R26, R26 to R27, R25 to R28
Changed lines of the file:
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@@
 		(on_board yes)
 		(dnp no)
-		(property "Reference" "#PWR056"
+		(property "Reference" "#PWR065"
 			(at 160.02 104.14 0)
 			(hide yes)
@@
 			(project "TurtlePico-Minimal"
 				(path "/7af2d99d-e350-48e7-86b4-20911ea922f3/3559871a-0f23-4a86-a659-f5f50e9db57b"
-					(reference "#PWR056")
+					(reference "#PWR065")
 					(unit 1)
 				)
@@
 		(on_board yes)
 		(dnp no)
-		(property "Reference" "Q4"
+		(property "Reference" "Q3"
 			(at 146.685 114.3 0)
 			(effects
@@
 			(project "TurtlePico-Minimal"
 				(path "/7af2d99d-e350-48e7-86b4-20911ea922f3/3559871a-0f23-4a86-a659-f5f50e9db57b"
-					(reference "Q4")
+					(reference "Q3")
 					(unit 1)
 				)
@@
 		(on_board yes)
 		(dnp no)
-		(property "Reference" "#PWR057"
+		(property "Reference" "#PWR068"
 			(at 187.96 107.95 0)
 			(hide yes)
@@
 			(project "TurtlePico-Minimal"
 				(path "/7af2d99d-e350-48e7-86b4-20911ea922f3/3559871a-0f23-4a86-a659-f5f50e9db57b"
-					(reference "#PWR057")
+					(reference "#PWR068")
 					(unit 1)
 				)
@@
 		(on_board yes)
 		(dnp no)
-		(property "Reference" "#PWR073"
+		(property "Reference" "#PWR067"
 			(at 167.64 133.35 0)
 			(hide yes)
@@
 			(project "TurtlePico-Minimal"
 				(path "/7af2d99d-e350-48e7-86b4-20911ea922f3/3559871a-0f23-4a86-a659-f5f50e9db57b"
-					(reference "#PWR073")
+					(reference "#PWR067")
 					(unit 1)
 				)
@@
 		(on_board yes)
 		(dnp no)
-		(property "Reference" "Q3"
+		(property "Reference" "Q2"
 			(at 119.38 113.03 0)
 			(effects
@@
 			(project "TurtlePico-Minimal"
 				(path "/7af2d99d-e350-48e7-86b4-20911ea922f3/3559871a-0f23-4a86-a659-f5f50e9db57b"
-					(reference "Q3")
+					(reference "Q2")
 					(unit 1)
 				)
@@
 		(on_board yes)
 		(dnp no)
-		(property "Reference" "#PWR026"
+		(property "Reference" "#PWR066"
 			(at 167.64 120.65 0)
 			(hide yes)
@@
 			(project "TurtlePico-Minimal"
 				(path "/7af2d99d-e350-48e7-86b4-20911ea922f3/3559871a-0f23-4a86-a659-f5f50e9db57b"
-					(reference "#PWR026")
+					(reference "#PWR066")
 					(unit 1)
 				)
@@
 		(on_board yes)
 		(dnp no)
-		(property "Reference" "R27"
+		(property "Reference" "R25"
 			(at 116.84 121.92 90)
 			(effects
@@
 			(project "TurtlePico-Minimal"
 				(path "/7af2d99d-e350-48e7-86b4-20911ea922f3/3559871a-0f23-4a86-a659-f5f50e9db57b"
-					(reference "R27")
+					(reference "R25")
 					(unit 1)
 				)
@@
 		(on_board yes)
 		(dnp no)
-		(property "Reference" "D4"
+		(property "Reference" "D3"
 			(at 115.57 106.68 90)
 			(effects
@@
 			(project "TurtlePico-Minimal"
 				(path "/7af2d99d-e350-48e7-86b4-20911ea922f3/3559871a-0f23-4a86-a659-f5f50e9db57b"
-					(reference "D4")
+					(reference "D3")
 					(unit 1)
 				)
@@
 		(on_board yes)
 		(dnp no)
-		(property "Reference" "J11"
+		(property "Reference" "J12"
 			(at 146.05 97.79 0)
 			(effects
@@
 			(project "TurtlePico-Minimal"
 				(path "/7af2d99d-e350-48e7-86b4-20911ea922f3/3559871a-0f23-4a86-a659-f5f50e9db57b"
-					(reference "J11")
+					(reference "J12")
 					(unit 1)
 				)
@@
 		(on_board yes)
 		(dnp no)
-		(property "Reference" "R26"
+		(property "Reference" "R27"
 			(at 130.81 114.3 90)
 			(effects
@@
 			(project "TurtlePico-Minimal"
 				(path "/7af2d99d-e350-48e7-86b4-20911ea922f3/3559871a-0f23-4a86-a659-f5f50e9db57b"
-					(reference "R26")
+					(reference "R27")
 					(unit 1)
 				)
@@
 			)
 		)
-		(property "Footprint" ""
+		(property "Footprint" "Package_DIP:DIP-8_W7.62mm"
 			(at 198.12 111.76 0)
 			(hide yes)
@@
 		(on_board yes)
 		(dnp no)
-		(property "Reference" "R24"
+		(property "Reference" "R26"
 			(at 121.92 106.68 90)
 			(effects
@@
 			(project "TurtlePico-Minimal"
 				(path "/7af2d99d-e350-48e7-86b4-20911ea922f3/3559871a-0f23-4a86-a659-f5f50e9db57b"
-					(reference "R24")
+					(reference "R26")
 					(unit 1)
 				)
@@
 		(on_board yes)
 		(dnp no)
-		(property "Reference" "#PWR055"
+		(property "Reference" "#PWR063"
 			(at 127 99.06 0)
 			(hide yes)
@@
 			(project "TurtlePico-Minimal"
 				(path "/7af2d99d-e350-48e7-86b4-20911ea922f3/3559871a-0f23-4a86-a659-f5f50e9db57b"
-					(reference "#PWR055")
+					(reference "#PWR063")
 					(unit 1)
 				)
@@
 		(on_board yes)
 		(dnp no)
-		(property "Reference" "J10"
+		(property "Reference" "J11"
 			(at 128.27 97.79 0)
 			(effects
@@
 			(project "TurtlePico-Minimal"
 				(path "/7af2d99d-e350-48e7-86b4-20911ea922f3/3559871a-0f23-4a86-a659-f5f50e9db57b"
-					(reference "J10")
+					(reference "J11")
 					(unit 1)
 				)
@@
 			)
 		)
-		(property "Footprint" ""
+		(property "Footprint" "Potentiometer_THT:Potentiometer_Bourns_3339P_Vertical_HandSoldering"
 			(at 167.64 121.92 0)
 			(hide yes)
@@
 		(on_board yes)
 		(dnp no)
-		(property "Reference" "#PWR059"
+		(property "Reference" "#PWR064"
 			(at 144.78 127 0)
 			(hide yes)
@@
 			(project "TurtlePico-Minimal"
 				(path "/7af2d99d-e350-48e7-86b4-20911ea922f3/3559871a-0f23-4a86-a659-f5f50e9db57b"
-					(reference "#PWR059")
+					(reference "#PWR064")
 					(unit 1)
 				)
@@
 		(on_board yes)
 		(dnp no)
-		(property "Reference" "R25"
+		(property "Reference" "R28"
 			(at 139.7 106.68 90)
 			(effects
@@
 			(project "TurtlePico-Minimal"
 				(path "/7af2d99d-e350-48e7-86b4-20911ea922f3/3559871a-0f23-4a86-a659-f5f50e9db57b"
-					(reference "R25")
+					(reference "R28")
 					(unit 1)
 				)
@@
 		(on_board yes)
 		(dnp no)
-		(property "Reference" "D3"
+		(property "Reference" "D4"
 			(at 130.81 106.68 90)
 			(effects
@@
 			(project "TurtlePico-Minimal"
 				(path "/7af2d99d-e350-48e7-86b4-20911ea922f3/3559871a-0f23-4a86-a659-f5f50e9db57b"
-					(reference "D3")
-					(unit 1)
-				)
+					(reference "D4")
+					(unit 1)
+				)
