File: board/advanced/Storage.kicad_sch (KiCad schematic)
At the start: 1 part, among them J1 Micro_SD

Commit message: put footprints and change schematics
Parts:
- J1: footprint Connector_Card:microSD_HC_Hirose_DM3D-SF -> Connector_Card:microSD_HC_Hirose_DM3AT-SF-PEJM5
Changed lines of the file:
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@@
 			)
 		)
-		(property "Footprint" "Connector_Card:microSD_HC_Hirose_DM3D-SF"
+		(property "Footprint" "Connector_Card:microSD_HC_Hirose_DM3AT-SF-PEJM5"
 			(at 203.2 92.71 0)
 			(hide yes)
