File: board/advanced/RP2350B.kicad_sch (KiCad schematic)
At the start: 40 parts, among them SW1 SW_Bootsel, U1 RP2350B-QFN80, U2 W25Q128JVS, U3 AP63203WU, Y1 ABM8-272-T3

Commit message: put footprints and change schematics
Parts:
- removed R6, R7: 27, Resistor_SMD:R_0603_1608Metric, symbol Device:R
- R1, R2, R3, R4, R5: footprint Resistor_SMD:R_0603_1608Metric -> Resistor_SMD:R_0201_0603Metric
- R6: renamed from R8; footprint Resistor_SMD:R_0603_1608Metric -> Resistor_SMD:R_0402_1005Metric
- R7: renamed from R9; footprint Resistor_SMD:R_0603_1608Metric -> Resistor_SMD:R_0402_1005Metric
- R8: renamed from R10; footprint Resistor_SMD:R_0603_1608Metric -> Resistor_SMD:R_0402_1005Metric
- R9: renamed from R11; footprint Resistor_SMD:R_0603_1608Metric -> Resistor_SMD:R_0402_1005Metric
Connections:
- net I/O_{0}: now also U1.40 (GPIO32); no longer U1.43 (GPIO34)
- net I/O_{10}: now also U1.54 (GPIO43_ADC3); no longer U1.56 (GPIO45_ADC5)
- net I/O_{11}: now also U1.55 (GPIO44_ADC4); no longer U1.57 (GPIO46_ADC6)
- net I/O_{12}: now also U1.56 (GPIO45_ADC5); no longer U1.58 (GPIO47_ADC7)
- net I/O_{1}: now also U1.42 (GPIO33); no longer U1.44 (GPIO35)
- net I/O_{2}: now also U1.43 (GPIO34); no longer U1.45 (GPIO36)
- net I/O_{3}: now also U1.44 (GPIO35); no longer U1.46 (GPIO37)
- net I/O_{4}: now also U1.45 (GPIO36); no longer U1.47 (GPIO38)
- net I/O_{5}: now also U1.46 (GPIO37); no longer U1.48 (GPIO39)
- net I/O_{6}: now also U1.47 (GPIO38); no longer U1.52 (GPIO41_ADC1)
- net I/O_{7}: now also U1.48 (GPIO39); no longer U1.53 (GPIO42_ADC2)
- net I/O_{8}: now also U1.52 (GPIO41_ADC1); no longer U1.54 (GPIO43_ADC3)
- net I/O_{9}: now also U1.53 (GPIO42_ADC2); no longer U1.55 (GPIO44_ADC4)
- net Echo renamed Echo/UART_{TX}
- net TRIG renamed TRIG/UART_{RX}
- new net I/O_{13}: U1.57 (GPIO46_ADC6)
- new net I/O_{14}: U1.58 (GPIO47_ADC7)

Commit message: change schematics and complete wiring
Parts:
- added R9: 10k, C_0402_1005Metric_small_pads:C_0402_1005Metric_small_pads, symbol Device:R
- added SW2: SW_Reset, SW_SKRPACE010:SW_SKRPACE010, symbol Switch:SW_Push
- C1, C10, C11, C12, C13, C14, C15, C17, C18, C19, C2, C20, C3, C4, C5, C6, C7, C8, C9: footprint Capacitor_SMD:C_0201_0603Metric -> C_0402_1005Metric_small_pads:C_0402_1005Metric_small_pads
- C16: footprint Capacitor_SMD:C_1206_3216Metric -> Capacitor_SMD:C_0603_1608Metric
- C21, C22: footprint Capacitor_SMD:C_0402_1005Metric -> C_0402_1005Metric_small_pads:C_0402_1005Metric_small_pads
- R1, R2, R3, R4, R5: footprint Resistor_SMD:R_0201_0603Metric -> C_0402_1005Metric_small_pads:C_0402_1005Metric_small_pads
- R10: renamed from R9; footprint Resistor_SMD:R_0402_1005Metric -> C_0402_1005Metric_small_pads:C_0402_1005Metric_small_pads
- R6, R7, R8: footprint Resistor_SMD:R_0402_1005Metric -> C_0402_1005Metric_small_pads:C_0402_1005Metric_small_pads
- U1: footprint Package_DFN_QFN:QFN-80-1EP_10x10mm_P0.4mm_EP3.4x3.4mm_ThermalVias -> RP2350_80QFN_minimal:RP2350-QFN-80-1EP_10x10_P0.4mm_EP3.4x3.4mm_ThermalVias
Connections:
- net Display_{BL}: now also U1.11 (GPIO12); no longer U1.38 (GPIO30)
- net Display_{DC}: now also U1.7 (GPIO9); no longer U1.3 (GPIO6)
- net Display_{RST}: now also U1.6 (GPIO8); no longer U1.2 (GPIO5)
- net ESC_{FR}: now also U1.39 (GPIO31); no longer U1.36 (GPIO28)
- net ESC_{RL}: now also U1.22 (GPIO22); no longer U1.12 (GPIO13)
- net ESC_{RR}: now also U1.36 (GPIO28); no longer U1.16 (GPIO16)
- net GND: now also SW2.1
- net I2S_{SCK}: now also U1.1 (GPIO4); no longer U1.19 (GPIO19)
- net I2S_{SD}: now also U1.3 (GPIO6); no longer U1.21 (GPIO21)
- net I2S_{WS}: now also U1.2 (GPIO5); no longer U1.20 (GPIO20)
- net LED_{L}: now also U1.16 (GPIO16); no longer U1.1 (GPIO4)
- net LED_{R}: now also U1.37 (GPIO29); no longer U1.18 (GPIO18)
- net MOTOR_A_{EN}: now also U1.25 (GPIO24); no longer U1.13 (GPIO14)
- net MOTOR_A_{IN}: now also U1.23 (GPIO23); no longer U1.17 (GPIO17)
- net MOTOR_B_{EN}: now also U1.27 (GPIO26); no longer U1.37 (GPIO29)
- net MOTOR_B_{IN}: now also U1.26 (GPIO25); no longer U1.14 (GPIO15)
- net SD_{CS}: now also U1.38 (GPIO30); no longer U1.28 (GPIO27)
- net SPI_{MISO}: now also U1.12 (GPIO13); no longer U1.11 (GPIO12)
- net SPI_{MOSI}: now also U1.8 (GPIO10); no longer U1.9 (GPIO11)
- net SPI_{SCK}: now also U1.9 (GPIO11); no longer U1.8 (GPIO10)
- net SW_{DIP}1: now also U1.20 (GPIO20); no longer U1.23 (GPIO23)
- net SW_{DIP}2: now also U1.19 (GPIO19); no longer U1.25 (GPIO24)
- net SW_{DIP}3: now also U1.18 (GPIO18); no longer U1.26 (GPIO25)
- net SW_{DIP}4: now also U1.17 (GPIO17); no longer U1.27 (GPIO26)
- net SW_{R}: now also U1.28 (GPIO27); no longer U1.22 (GPIO22)
- net TOUCH_{CS}: now also U1.21 (GPIO21); no longer U1.39 (GPIO31)
- net RUN: now reaches U1.35 (RUN)
- net RUN: now also R9.2
- net at R4.1: now also U1.13 (GPIO14); no longer U1.6 (GPIO8)
- net at R5.1: now also U1.14 (GPIO15); no longer U1.7 (GPIO9)
- net D+0 renamed D+
- net D-0 renamed D-
- new net: R9.1, SW2.2
- no-connect marks 1 -> 0
Other:
- moved on the sheet: R4, R5, R6, R7

Commit message: add LTB example and more
Parts:
- C1, C2, C4, C6: Mouser Part Number (none) -> 81-GRM155R60J475ME7J; Mouser Price/Stock (none) -> https://www.mouser.jp/ProductDetail/Murata-Electronics/GRM1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
- C10, C11, C12, C13, C14, C15, C17, C20, C3, C5, C7, C8, C9: Mouser Part Number (none) -> 81-GRM15R61A104KA01J; Mouser Price/Stock (none) -> https://www.mouser.jp/ProductDetail/Murata-Electronics/GRM1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
- C16: Mouser Part Number (none) -> 81-GRM188C81C106MA3D; Mouser Price/Stock (none) -> https://www.mouser.jp/ProductDetail/Murata-Electronics/GRM1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
- C18, C19: Mouser Part Number (none) -> 81-GRT1555C1E150JA2D; Mouser Price/Stock (none) -> https://www.mouser.jp/ProductDetail/Murata-Electronics/GRT1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
- C21, C22: Mouser Part Number (none) -> 81-GRM155R60J226ME1D; Mouser Price/Stock (none) -> https://www.mouser.jp/ProductDetail/Murata-Electronics/GRM1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
- L1: Mouser Part Number (none) -> 815-AB201610S3R3101T; Mouser Price/Stock (none) -> https://www.mouser.jp/ProductDetail/ABRACON/AOTA-B201610S3R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
- L2: Mouser Part Number (none) -> 815-AOTB201610S4R7MT; Mouser Price/Stock (none) -> https://www.mouser.jp/ProductDetail/ABRACON/AOTA-B201610S4R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
- R1, R4, R5: Mouser Part Number (none) -> 667-ERJ-2GEJ330X; Mouser Price/Stock (none) -> https://www.mouser.jp/ProductDetail/Panasonic/ERJ-2GEJ330X?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
- R10, R8: Mouser Part Number (none) -> 667-ERJ-2GEJ102X; Mouser Price/Stock (none) -> https://www.mouser.jp/ProductDetail/Panasonic/ERJ-2GEJ102X?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
- R2, R3: Mouser Part Number (none) -> 667-ERJ-2GEJ270X; Mouser Price/Stock (none) -> https://www.mouser.jp/ProductDetail/Panasonic/ERJ-2GEJ270X?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
- R6, R7: Mouser Part Number (none) -> 667-ERJ-2RKF4701X; Mouser Price/Stock (none) -> https://www.mouser.jp/ProductDetail/Panasonic/ERJ-2RKF4701X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
- R9: Mouser Part Number (none) -> 667-ERJ-2GEJ103X; Mouser Price/Stock (none) -> https://www.mouser.jp/ProductDetail/Panasonic/ERJ-2GEJ103X?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
- SW1, SW2: Mouser Part Number (none) -> 688-SKRPACE010; Mouser Price/Stock (none) -> https://www.mouser.jp/ProductDetail/Alps-Alpine/SKRPACE010?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
- U1: Mouser Part Number (none) -> 358-SC1510; Mouser Price/Stock (none) -> https://www.mouser.jp/ProductDetail/Raspberry-Pi/SC1510?qs=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
- U2: Mouser Part Number (none) -> 454-W25Q128JVSIQTR; Mouser Price/Stock (none) -> https://www.mouser.jp/ProductDetail/Winbond/W25Q128JVSIQ-TR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
- U3: Mouser Part Number (none) -> 621-AP63203WU-7; Mouser Price/Stock (none) -> https://www.mouser.jp/ProductDetail/Diodes-Incorporated/AP6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
- Y1: Mouser Part Number (none) -> 815-ABM8-272-T3; Mouser Price/Stock (none) -> https://www.mouser.jp/ProductDetail/ABRACON/ABM8-272-T3?qs=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
