File: board/advanced/TurtlePico-Leatherback.kicad_pcb (KiCad board)
At the start: 2 copper layers, 63.5 x 69.3 mm, 127 parts, among them J1 Micro_SD, J10 AudioJack3, J11 LED_{R}, J12 LED_{L}, J13 UltraSonic, J14 Debug, J15 Display, J16 TouchDisplay, J17 Conn_02x09_Odd_Even, J2 USB_C_Receptacle_USB2.0_16P, J3 Jack-DC, J4 RMotor, J5 LMotor, J6 FR_ESC, J7 FL_ESC, J8 RR_ESC, J9 RL_ESC, Q1 DMP6050SSD, Q2 2SC4213, Q3 2SC4213, SW1 SW_Bootsel, SW2 SW_Reset, SW3 SW_{R}, SW4 SW_{L}, SW5 SW_DIP_x04, U1 RP2350B-QFN80, U2 W25Q128JVS, U3 AP63203WU, U4 CYPD3177-24LQ, U5 DRV8835DSSR, U6 INA260, U7 BNO086, U8 BME280, U9 PCM5102A, Y1 ABM8-272-T3, Y2 ABS06-32.768KHZ-T

Commit message: add v1.2 model
Parts:
- moved G2 5.33 mm to (210.6, 125.5)
Other:
- board text added: "Powered by"
