File: board/main/TurtlePico.kicad_pcb (KiCad board)
At the start: 2 copper layers, 63.5 x 69.3 mm, 46 parts, among them IC1 DRV8835DSSR, J1 USB-C, J10 LMotor, J11 Micro_SD, J12 FR_ESC, J13 FL_ESC, J14 RR_ESC, J15 RL_ESC, J2 AudioJack3, J3 LED, J4 LED, J5 9DoF, J6 Temperature, J7 UltraSonic, J8 OLED, J9 RMotor, Q1 2SC4213, Q2 2SC4213, SW1 SW_Push, SW2 SW_Push, U1 PCM5102A, U2 Pico

Commit message: add v1.2 model
Parts:
- removed the G*** at (145.8, 73.7)
- added G***: LOGO, JinPro:JinNeuron_Logo, B.Cu at (146.7, 88.4)
- added G***: LOGO, TurtlePico:TurtlePico, B.Cu at (145.8, 75.2)
- moved G*** 16.0 mm to (158.5, 69.1)
Routing:
- net +5V: track 14.3 -> 13.8 mm
Other:
- board text added: "Powered by"
- board text added: "v1.2"
- board text removed: "Turtle Pico v1.1"
